Commit message: Update robot_description.urdf.xacro

File: urdf/robot_description.urdf.xacro (robot description, xacro)
@@ -2,4 +2,5 @@
 <robot name="applebot" xmlns:xacro="http://ros.org/wiki/xacro">
     <xacro:include filename="$(find applebot)/urdf/common_macros.xacro" />
+    <xacro:include filename="$(find applebot)/urdf/robot_control.gazebo.xacro" />
     <!-- <gazebo>
         <static>true</static>
@@ -25,10 +26,10 @@
         </visual>
         <collision>
-            <origin xyz="0 0 0" rpy="0 0 0"/>
+            <origin xyz="0.3 -0.5 0.2" rpy="0 0 0"/>
             <geometry>
-                <box size="1 0.600 0.350"/>
+                <box size="0.600 1 0.4"/>
             </geometry>
         </collision>
-        <xacro:inertial_box length="1" width="0.600" height="0.350" density="${density_pla}">
+        <xacro:inertial_box length="0.600" width="1" height="0.350" density="${density_pla}">
             <origin xyz="0 0 0" rpy="0 0 0"/>
         </xacro:inertial_box>
@@ -52,7 +53,7 @@
         </visual>
         <collision>
-            <origin xyz="0 0 0" rpy="0 0 0"/>
+            <origin xyz="0 0 0.04" rpy="0 0 0"/>
             <geometry>
-                <cylinder length="0.1" radius="0.1" />
+                <cylinder length="0.08" radius="0.1" />
             </geometry>
         </collision>
@@ -79,7 +80,7 @@
         </visual>
         <collision>
-            <origin xyz="0 0 0" rpy="0 0 0"/>
+            <origin xyz="0 0 0.04" rpy="0 0 0"/>
             <geometry>
-                <cylinder length="0.1" radius="0.1" />
+                <cylinder length="0.08" radius="0.1" />
             </geometry>
         </collision>
@@ -106,7 +107,7 @@
         </visual>
         <collision>
-            <origin xyz="0 0 0" rpy="0 0 0"/>
+            <origin xyz="0 0 0.04" rpy="0 0 0"/>
             <geometry>
-                <cylinder length="0.1" radius="0.1" />
+                <cylinder length="0.08" radius="0.1" />
             </geometry>
         </collision>
@@ -133,7 +134,7 @@
         </visual>
         <collision>
-            <origin xyz="0 0 0" rpy="0 0 0"/>
+            <origin xyz="0 0 0.04" rpy="0 0 0"/>
             <geometry>
-                <cylinder length="0.1" radius="0.1" />
+                <cylinder length="0.08" radius="0.1" />
             </geometry>
         </collision>

Commit message: Update robot_description.urdf.xacro

File: urdf/robot_description.urdf.xacro (robot description, xacro)
@@ -32,5 +32,5 @@
         </collision>
         <xacro:inertial_box length="0.600" width="1" height="0.350" density="${density_pla}">
-            <origin xyz="0 0 0" rpy="0 0 0"/>
+            <origin xyz="0.3 -0.5 0.2" rpy="0 0 0"/>
         </xacro:inertial_box>
     </link>
@@ -38,5 +38,5 @@
     <!-- ==================================== -->
     <joint type="continuous" name="front_left_wheel_joint">
-        <origin xyz="0 -0.100 0.100" rpy="-${pi/2} 0 ${pi/2}"/>
+        <origin xyz="0 -0.100 0" rpy="-${pi/2} 0 ${pi/2}"/>
         <child link="front_left_wheel_link"/>
         <parent link="mobile_base_link"/>
@@ -58,6 +58,6 @@
             </geometry>
         </collision>
-        <xacro:inertial_cylinder radius="0.1" length="0.1" density="${density_pla}">
-            <origin xyz="0 0 0" rpy="0 0 0"/>
+        <xacro:inertial_cylinder radius="0.08" length="0.1" density="${density_pla}">
+            <origin xyz="0 0 0.04" rpy="0 0 0"/>
         </xacro:inertial_cylinder>
     </link>
@@ -65,5 +65,5 @@
     <!-- ==================================== -->
     <joint type="continuous" name="front_right_wheel_joint">
-        <origin xyz="0.600 -0.099 0.100" rpy="-${pi/2} 0 -${pi/2}"/>
+        <origin xyz="0.600 -0.099 0" rpy="-${pi/2} 0 -${pi/2}"/>
         <child link="front_right_wheel_link"/>
         <parent link="mobile_base_link"/>
@@ -85,6 +85,6 @@
             </geometry>
         </collision>
-        <xacro:inertial_cylinder radius="0.1" length="0.1" density="${density_pla}">
-            <origin xyz="0 0 0" rpy="0 0 0"/>
+        <xacro:inertial_cylinder radius="0.08" length="0.1" density="${density_pla}">
+            <origin xyz="0 0 0.04" rpy="0 0 0"/>
         </xacro:inertial_cylinder>
     </link>
@@ -92,5 +92,5 @@
     <!-- ==================================== -->
     <joint type="continuous" name="back_right_wheel_joint">
-        <origin xyz="0.600 -0.900 0.100" rpy="-${pi/2} 0 -${pi/2}"/>
+        <origin xyz="0.600 -0.900 0" rpy="-${pi/2} 0 -${pi/2}"/>
         <child link="back_right_wheel_link"/>
         <parent link="mobile_base_link"/>
@@ -112,6 +112,6 @@
             </geometry>
         </collision>
-        <xacro:inertial_cylinder radius="0.1" length="0.1" density="${density_pla}">
-            <origin xyz="0 0 0" rpy="0 0 0"/>
+        <xacro:inertial_cylinder radius="0.08" length="0.1" density="${density_pla}">
+            <origin xyz="0 0 0.04" rpy="0 0 0"/>
         </xacro:inertial_cylinder>
     </link>
@@ -119,5 +119,5 @@
     <!-- ==================================== -->
     <joint type="continuous" name="back_left_wheel_joint">
-        <origin xyz="0 -0.900 0.100" rpy="-${pi/2} 0 ${pi/2}"/>
+        <origin xyz="0 -0.900 0" rpy="-${pi/2} 0 ${pi/2}"/>
         <child link="back_left_wheel_link"/>
         <parent link="mobile_base_link"/>
@@ -139,7 +139,34 @@
             </geometry>
         </collision>
-        <xacro:inertial_cylinder radius="0.1" length="0.1" density="${density_pla}">
-            <origin xyz="0 0 0" rpy="0 0 0"/>
+        <xacro:inertial_cylinder radius="0.08" length="0.1" density="${density_pla}">
+            <origin xyz="0 0 0.04" rpy="0 0 0"/>
         </xacro:inertial_cylinder>
     </link>
+    <!-- ARM BASE -->
+    <!-- ==================================== -->
+    <joint type="revolute" name="arm_base_joint">
+        <origin xyz="0.3 -0.5 0.3" rpy="0 0 -${pi/2}"/>
+        <child link="arm_base_link"/>
+        <parent link="mobile_base_link"/>
+        <axis xyz="0 0 1" rpy="0 0 0"/>
+        <limit effort="100" velocity="100" lower="-${pi}" upper="${pi}"/>
+        <dynamics damping="0.7" friction="1.0"/>
+    </joint>
+    <link name="arm_base_link">
+        <visual>
+            <origin xyz="0 0 0" rpy="0 0 0"/>
+            <geometry>
+                <mesh filename="$(find applebot)/meshes/armiiiii.stl" />
+            </geometry>
+        </visual>
+        <collision>
+            <origin xyz="0.3 -0.5 0.2" rpy="0 0 0"/>
+            <geometry>
+                <box size="0.600 1 0.4"/>
+            </geometry>
+        </collision>
+        <xacro:inertial_box length="0.600" width="1" height="0.350" density="0.00001">
+            <origin xyz="0.3 -0.5 0.2" rpy="0 0 0"/>
+        </xacro:inertial_box>
+    </link>
 </robot>

Commit message: Update robot_description.urdf.xacro

File: urdf/robot_description.urdf.xacro (robot description, xacro)
@@ -6,5 +6,6 @@
         <static>true</static>
     </gazebo> -->
-    <xacro:property name="density_pla" value="600" />
+    <xacro:property name="density_pla" value="100" />
+    <xacro:property name="friction_wheels" value="100" />
     <!--############################### -->
     <!-- MOBILE PLATFORM -->
@@ -43,5 +44,5 @@
         <axis xyz="0 0 1" rpy="0 0 0"/>
         <limit effort="1000" velocity="1000"/>
-        <dynamics damping="0.7" friction="1.0"/>
+        <dynamics damping="0.7" friction="${friction_wheels}"/>
     </joint>
     <link name="front_left_wheel_link">
@@ -65,10 +66,10 @@
     <!-- ==================================== -->
     <joint type="continuous" name="front_right_wheel_joint">
-        <origin xyz="0.600 -0.099 0" rpy="-${pi/2} 0 -${pi/2}"/>
+        <origin xyz="0.600 -0.100 0" rpy="-${pi/2} 0 -${pi/2}"/>
         <child link="front_right_wheel_link"/>
         <parent link="mobile_base_link"/>
         <axis xyz="0 0 1" rpy="0 0 0"/>
         <limit effort="1000" velocity="1000"/>
-        <dynamics damping="0.7" friction="1.0"/>
+        <dynamics damping="0.7" friction="${friction_wheels}"/>
     </joint>
     <link name="front_right_wheel_link">
@@ -97,5 +98,5 @@
         <axis xyz="0 0 1" rpy="0 0 0"/>
         <limit effort="1000" velocity="1000"/>
-        <dynamics damping="0.7" friction="1.0"/>
+        <dynamics damping="0.7" friction="${friction_wheels}"/>
     </joint>
     <link name="back_right_wheel_link">
@@ -124,5 +125,5 @@
         <axis xyz="0 0 1" rpy="0 0 0"/>
         <limit effort="1000" velocity="1000"/>
-        <dynamics damping="0.7" friction="1.0"/>
+        <dynamics damping="0.7" friction="${friction_wheels}"/>
     </joint>
     <link name="back_left_wheel_link">
@@ -161,5 +162,5 @@
         </visual>
         <collision>
-            <origin xyz="0.3 -0.5 0.2" rpy="0 0 0"/>
+            <origin xyz="0 0 0.3" rpy="0 0 ${pi/2}"/>
             <geometry>
                 <box size="0.600 1 0.4"/>
